File: sensor_system/sensor_system.kicad_pcb (KiCad board)
At the start: 2 copper layers, 137.1 x 28.8 mm, 58 parts, among them J1 Magnetic connector, J2 Solar_panels, Q1 SBC817, Q2 MJD45H11, SW1 SW_DPDT_x2, U1 TLC555xD, U2 XC6206PxxxMR, U3 MCP73833, U4 BME280, U5 ESP32-DEVKIT-V1, U7 TPS63002

Commit message: Final board
Parts:
- moved R15 1.11 mm to (144.8, 26.1)
- moved C14 0.65 mm to (103.9, 45.2)
- moved C15 0.39 mm to (105.9, 45.2)
- moved R1 0.26 mm to (97.0, 43.8)
- moved C9 0.15 mm to (151.1, 33.4)
- moved C10 0.06 mm to (105.5, 42.0)
- moved C3 0.05 mm to (96.9, 45.8)
Routing:
- net Net-(D3-K): track 21.9 -> 36.3 mm
- net /power_supply/5V: track 13.8 -> 0.95 mm, vias 1 -> 0
- net Net-(BT1-+): track 17.1 -> 28.8 mm
- net Net-(Q2-E): track 7.86 -> 16.5 mm
- net 3V: track 6.24 -> 0.00 mm
- net Net-(D3-A): track 5.83 -> 11.3 mm
- net Net-(D10-A): track 41.6 -> 46.4 mm
- net Net-(U1-THR): track 18.0 -> 17.0 mm
- net Soil: vias 0 -> 1
- net Earth: vias 1 -> 17
- added copper zone on F.Cu, net /power_supply/5V
- added copper zone on B.Cu, net 3V

Commit message: Final board fix
Routing:
- net /power_supply/5V: track 0.95 -> 1.70 mm
Changed lines of the file:
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@@
   (segment (start 110.8 47.2) (end 110.8 46.75) (width 0.7) (layer "F.Cu") (net 6))
   (segment (start 108 47.25) (end 108 46.75) (width 0.7) (layer "F.Cu") (net 6))
+  (segment (start 108 46.75) (end 107.25 46.75) (width 0.7) (layer "F.Cu") (net 6))
   (segment (start 111.7875 39.45) (end 108.85 39.45) (width 0.5) (layer "F.Cu") (net 7))
   (segment (start 148.4375 36.45) (end 148.4375 40.9) (width 0.7) (layer "F.Cu") (net 8))
@@
         (xy 102.65 52.7)
         (xy 102.65 45.3)
-        (xy 111.45 45.25)
-        (xy 111.45 48.2)
+        (xy 111.55 45.25)
+        (xy 111.55 48.2)
         (xy 105.9 48.2)
         (xy 105.9 52.7)

Commit message: Gala versija
Parts:
- added TP1: TestPoint, Connector_PinHeader_1.00mm:PinHeader_1x01_P1.00mm_Vertical, F.Cu at (123.5, 35.4)
- moved BT1 0.15 mm to (134.8, 35.0)
- moved TH1 0.15 mm to (138.0, 35.0)
Routing:
- net Net-(D10-A): track 46.4 -> 49.8 mm
