File: sensor_system/sensor_system.kicad_sch (KiCad schematic)
At the start: 8 parts, among them U4 BME280, U5 ESP32-DEVKIT-V1

Commit message: Board V2
Parts:
- C11, C12: footprint (none) -> Capacitor_SMD:C_0805_2012Metric
- R15, R17: footprint (none) -> Resistor_SMD:R_0805_2012Metric
Connections:
- net Soil: now also U5.28 (D13); no longer U5.21 (D32)
- net at D9.2 (A), R13.1: now also U5.19 (D34); no longer U5.5 (D4)
Other:
- moved on the sheet: D9, R13
Changed lines of the file:
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@@
 (kicad_sch (version 20230121) (generator eeschema)
   (paper "A4")
-  (junction (at 60.96 60.96) (diameter 0) (color 0 0 0 0)
+  (junction (at 109.22 73.66) (diameter 0) (color 0 0 0 0)
   )
   (junction (at 102.87 81.28) (diameter 0) (color 0 0 0 0)
@@
   (no_connect (at 72.39 60.96))
   (no_connect (at 102.87 55.88))
-  (no_connect (at 72.39 63.5))
+  (no_connect (at 102.87 66.04))
   (no_connect (at 102.87 40.64))
   (no_connect (at 102.87 63.5))
@@
   (no_connect (at 72.39 66.04))
   (no_connect (at 102.87 38.1))
-  (no_connect (at 102.87 73.66))
+  (no_connect (at 72.39 55.88))
   (no_connect (at 72.39 71.12))
   (no_connect (at 72.39 40.64))
@@
     (stroke (width 0) (type default))
   )
-  (wire (pts (xy 63.5 55.88) (xy 72.39 55.88))
-    (stroke (width 0) (type default))
-  )
   (wire (pts (xy 55.88 43.18) (xy 62.23 43.18))
     (stroke (width 0) (type default))
@@
     (stroke (width 0) (type default))
   )
-  (wire (pts (xy 63.5 60.96) (xy 60.96 60.96))
-    (stroke (width 0) (type default))
-  )
   (wire (pts (xy 102.87 82.55) (xy 102.87 81.28))
     (stroke (width 0) (type default))
   )
+  (wire (pts (xy 102.87 73.66) (xy 109.22 73.66))
+    (stroke (width 0) (type default))
+  )
   (wire (pts (xy 102.87 78.74) (xy 102.87 81.28))
     (stroke (width 0) (type default))
   )
   (wire (pts (xy 146.05 63.5) (xy 146.05 54.61))
-    (stroke (width 0) (type default))
-  )
-  (wire (pts (xy 63.5 55.88) (xy 63.5 60.96))
     (stroke (width 0) (type default))
   )
@@
     )
   )
-  (global_label "3V3" (shape input) (at 60.96 53.34 90) (fields_autoplaced)
+  (global_label "3V3" (shape input) (at 109.22 66.04 90) (fields_autoplaced)
     (effects (font (size 1.27 1.27)) (justify left))
-    (property "Intersheetrefs" "${INTERSHEET_REFS}" (at 60.96 46.9266 90)
+    (property "Intersheetrefs" "${INTERSHEET_REFS}" (at 109.22 59.6266 90)
       (effects (font (size 1.27 1.27)) (justify left) hide)
     )
@@
     )
   )
-  (global_label "Soil" (shape input) (at 102.87 66.04 0) (fields_autoplaced)
-    (effects (font (size 1.27 1.27)) (justify left))
-    (property "Intersheetrefs" "${INTERSHEET_REFS}" (at 109.4043 66.04 0)
-      (effects (font (size 1.27 1.27)) (justify left) hide)
+  (global_label "Soil" (shape input) (at 72.39 63.5 180) (fields_autoplaced)
+    (effects (font (size 1.27 1.27)) (justify right))
+    (property "Intersheetrefs" "${INTERSHEET_REFS}" (at 65.8557 63.5 0)
+      (effects (font (size 1.27 1.27)) (justify right) hide)
     )
   )
@@
     )
   )
-  (symbol (lib_id "Device:D_Photo") (at 60.96 58.42 270) (unit 1)
-    (in_bom yes) (on_board yes) (dnp no) (fields_autoplaced)
-    (property "Reference" "D9" (at 68.58 57.4675 0)
-      (effects (font (size 1.27 1.27)))
-    )
-    (property "Value" "D_Photo" (at 66.04 57.4675 0)
-      (effects (font (size 1.27 1.27)))
-    )
-    (property "Footprint" "LED_THT:LED_D5.0mm" (at 60.96 57.15 0)
-      (effects (font (size 1.27 1.27)) hide)
-    )
-    (property "Datasheet" "~" (at 60.96 57.15 0)
+  (symbol (lib_id "Device:D_Photo") (at 109.22 71.12 270) (unit 1)
+    (in_bom yes) (on_board yes) (dnp no) (fields_autoplaced)
+    (property "Reference" "D9" (at 116.84 70.1675 0)
+      (effects (font (size 1.27 1.27)))
+    )
+    (property "Value" "D_Photo" (at 114.3 70.1675 0)
+      (effects (font (size 1.27 1.27)))
+    )
+    (property "Footprint" "LED_THT:LED_D5.0mm" (at 109.22 69.85 0)
+      (effects (font (size 1.27 1.27)) hide)
+    )
+    (property "Datasheet" "~" (at 109.22 69.85 0)
       (effects (font (size 1.27 1.27)) hide)
     )
@@
       (effects (font (size 1.27 1.27)) (justify left))
     )
-    (property "Footprint" "" (at 144.272 67.31 90)
+    (property "Footprint" "Resistor_SMD:R_0805_2012Metric" (at 144.272 67.31 90)
       (effects (font (size 1.27 1.27)) hide)
     )
@@
       (effects (font (size 1.27 1.27)))
     )
-    (property "Footprint" "" (at 162.56 40.9448 0)
+    (property "Footprint" "Capacitor_SMD:C_0805_2012Metric" (at 162.56 40.9448 0)
       (effects (font (size 1.27 1.27)) hide)
     )
@@
       (effects (font (size 1.27 1.27)))
     )
-    (property "Footprint" "" (at 162.56 35.8648 0)
+    (property "Footprint" "Capacitor_SMD:C_0805_2012Metric" (at 162.56 35.8648 0)
       (effects (font (size 1.27 1.27)) hide)
     )
@@
       (effects (font (size 1.27 1.27)) (justify left))
     )
-    (property "Footprint" "" (at 137.922 67.31 90)
+    (property "Footprint" "Resistor_SMD:R_0805_2012Metric" (at 137.922 67.31 90)
       (effects (font (size 1.27 1.27)) hide)
     )
@@
     )
   )
-  (symbol (lib_id "Device:R") (at 60.96 64.77 0) (unit 1)
-    (in_bom yes) (on_board yes) (dnp no) (fields_autoplaced)
-    (property "Reference" "R13" (at 66.04 64.77 90)
-      (effects (font (size 1.27 1.27)))
-    )
-    (property "Value" "10k" (at 63.5 64.77 90)
-      (effects (font (size 1.27 1.27)))
-    )
-    (property "Footprint" "Resistor_SMD:R_0805_2012Metric" (at 59.182 64.77 90)
-      (effects (font (size 1.27 1.27)) hide)
-    )
-    (property "Datasheet" "~" (at 60.96 64.77 0)
+  (symbol (lib_id "Device:R") (at 109.22 77.47 0) (unit 1)
+    (in_bom yes) (on_board yes) (dnp no) (fields_autoplaced)
+    (property "Reference" "R13" (at 114.3 77.47 90)
+      (effects (font (size 1.27 1.27)))
+    )
+    (property "Value" "10k" (at 111.76 77.47 90)
+      (effects (font (size 1.27 1.27)))
+    )
+    (property "Footprint" "Resistor_SMD:R_0805_2012Metric" (at 107.442 77.47 90)
+      (effects (font (size 1.27 1.27)) hide)
+    )
+    (property "Datasheet" "~" (at 109.22 77.47 0)
       (effects (font (size 1.27 1.27)) hide)
     )
@@
     )
   )
-  (symbol (lib_id "power:Earth") (at 60.96 68.58 0) (unit 1)
-    (in_bom yes) (on_board yes) (dnp no) (fields_autoplaced)
-    (property "Reference" "#PWR016" (at 60.96 74.93 0)
-      (effects (font (size 1.27 1.27)) hide)
-    )
-    (property "Value" "Earth" (at 60.96 72.39 0)
-      (effects (font (size 1.27 1.27)) hide)
-    )
-    (property "Footprint" "" (at 60.96 68.58 0)
-      (effects (font (size 1.27 1.27)) hide)
-    )
-    (property "Datasheet" "~" (at 60.96 68.58 0)
-      (effects (font (size 1.27 1.27)) hide)
-    )
+  (symbol (lib_id "power:Earth") (at 109.22 81.28 0) (unit 1)
+    (in_bom yes) (on_board yes) (dnp no) (fields_autoplaced)
+    (property "Reference" "#PWR016" (at 109.22 87.63 0)
+      (effects (font (size 1.27 1.27)) hide)
+    )
+    (property "Value" "Earth" (at 109.22 85.09 0)
+      (effects (font (size 1.27 1.27)) hide)
+    )
+    (property "Footprint" "" (at 109.22 81.28 0)
+      (effects (font (size 1.27 1.27)) hide)
+    )
+    (property "Datasheet" "~" (at 109.22 81.28 0)
+      (effects (font (size 1.27 1.27)) hide)
+    )

Commit message: Board fix 2.0
Connections:
- net 3V3: now also D9.2 (A); no longer D9.1 (K)
- net at R13.1, U5.19 (D34): now also D9.1 (K); no longer D9.2 (A)
Other:
- moved on the sheet: D9
Changed lines of the file:
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@@
 (kicad_sch (version 20230121) (generator eeschema)
   (paper "A4")
+  (junction (at 102.87 81.28) (diameter 0) (color 0 0 0 0)
+  )
   (junction (at 109.22 73.66) (diameter 0) (color 0 0 0 0)
-  )
-  (junction (at 102.87 81.28) (diameter 0) (color 0 0 0 0)
   )
   (no_connect (at 72.39 60.96))
@@
     )
   )
-  (symbol (lib_id "Device:D_Photo") (at 109.22 71.12 270) (unit 1)
+  (symbol (lib_id "Device:D_Photo") (at 109.22 68.58 90) (unit 1)
     (in_bom yes) (on_board yes) (dnp no) (fields_autoplaced)
-    (property "Reference" "D9" (at 116.84 70.1675 0)
-      (effects (font (size 1.27 1.27)))
+    (property "Reference" "D9" (at 111.76 68.8975 90)
+      (effects (font (size 1.27 1.27)) (justify right))
     )
-    (property "Value" "D_Photo" (at 114.3 70.1675 0)
-      (effects (font (size 1.27 1.27)))
+    (property "Value" "D_Photo" (at 111.76 71.4375 90)
+      (effects (font (size 1.27 1.27)) (justify right))
     )
     (property "Footprint" "LED_THT:LED_D5.0mm" (at 109.22 69.85 0)

Commit message: Gala versija
Parts:
- removed D9: D_Photo, LED_THT:LED_D5.0mm, symbol Device:D_Photo
- added R18: R_Photo, symbol Device:R_Photo
Connections:
- net 3V3: now also R18.1
- net at R13.1, U5.19 (D34): now also R18.2
Changed lines of the file:
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@@
 (kicad_sch (version 20230121) (generator eeschema)
   (paper "A4")
+  (junction (at 109.22 73.66) (diameter 0) (color 0 0 0 0)
+  )
   (junction (at 102.87 81.28) (diameter 0) (color 0 0 0 0)
-  )
-  (junction (at 109.22 73.66) (diameter 0) (color 0 0 0 0)
   )
   (no_connect (at 72.39 60.96))
@@
     )
   )
-  (symbol (lib_id "Device:D_Photo") (at 109.22 68.58 90) (unit 1)
+  (symbol (lib_id "Device:R_Photo") (at 109.22 69.85 0) (unit 1)
     (in_bom yes) (on_board yes) (dnp no) (fields_autoplaced)
-    (property "Reference" "D9" (at 111.76 68.8975 90)
-      (effects (font (size 1.27 1.27)) (justify right))
+    (property "Reference" "R18" (at 111.76 69.215 0)
+      (effects (font (size 1.27 1.27)) (justify left))
     )
-    (property "Value" "D_Photo" (at 111.76 71.4375 90)
-      (effects (font (size 1.27 1.27)) (justify right))
+    (property "Value" "R_Photo" (at 111.76 71.755 0)
+      (effects (font (size 1.27 1.27)) (justify left))
     )
-    (property "Footprint" "LED_THT:LED_D5.0mm" (at 109.22 69.85 0)
-      (effects (font (size 1.27 1.27)) hide)
+    (property "Footprint" "" (at 110.49 76.2 90)
+      (effects (font (size 1.27 1.27)) (justify left) hide)
     )
-    (property "Datasheet" "~" (at 109.22 69.85 0)
+    (property "Datasheet" "~" (at 109.22 71.12 0)
       (effects (font (size 1.27 1.27)) hide)
     )
@@
       (project "sensor_system"
         (path "/d745cb62-8f4d-408c-9af8-25e31ee1e0d0"
-          (reference "D9") (unit 1)
+          (reference "R18") (unit 1)
         )
       )
